File: 7segmentos/7segmentos.sch (KiCad schematic (older format))
At the start: 31 parts, among them J1 AVR-ISP-6, J2 comunicação, J3 alimentacao, J4 digito_1, J5 digito_2, J6 digito_3, J7 digito_4, Q1 Si2319CDS, Q2 Si2319CDS, Q3 Si2319CDS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

Commit message: Desenvolvendo o esquemático
Parts:
- removed J1: AVR-ISP-6, Connector_PinSocket_2.54mm:PinSocket_1x06_P2.54mm_Vertical, symbol Connector:AVR-ISP-6
- added J1: ISP, Connector_PinSocket_2.54mm:PinSocket_1x06_P2.54mm_Vertical, symbol Connector_Generic:Conn_01x06
- added SW1: SW_Push_Dual, Button_Switch_THT:SW_TH_Tactile_Omron_B3F-10xx, symbol Switch:SW_Push_Dual
- C1, C2, C3, C4, C5, C6, C7: footprint Capacitor_THT:CP_Radial_D8.0mm_P5.00mm -> Capacitor_THT:CP_Radial_D6.3mm_P2.50mm
Connections:
- net +5V: now also J1.1 (Pin_1)
- net 1: now also J4.8 (Pin_8); no longer J4.1 (Pin_1)
- net 2: now also J5.8 (Pin_8); no longer J5.1 (Pin_1)
- net 3: now also J6.8 (Pin_8); no longer J6.1 (Pin_1)
- net 4: now also J7.8 (Pin_8); no longer J7.1 (Pin_1)
- net GND: now also J1.6 (Pin_6), SW1.4
- net a: now also J4.7 (Pin_7), J5.7 (Pin_7), J6.7 (Pin_7), J7.7 (Pin_7); no longer J4.8 (Pin_8), J5.8 (Pin_8), J6.8 (Pin_8), J7.8 (Pin_8)
- net b: now also J4.6 (Pin_6), J5.6 (Pin_6), J6.6 (Pin_6), J7.6 (Pin_6); no longer J4.7 (Pin_7), J5.7 (Pin_7), J6.7 (Pin_7), J7.7 (Pin_7)
- net c: now also J4.5 (Pin_5), J5.5 (Pin_5), J6.5 (Pin_5), J7.5 (Pin_5); no longer J4.6 (Pin_6), J5.6 (Pin_6), J6.6 (Pin_6), J7.6 (Pin_6)
- net d: now also J4.4 (Pin_4), J5.4 (Pin_4), J6.4 (Pin_4), J7.4 (Pin_4); no longer J4.5 (Pin_5), J5.5 (Pin_5), J6.5 (Pin_5), J7.5 (Pin_5)
- net e: now also J4.3 (Pin_3), J5.3 (Pin_3), J6.3 (Pin_3), J7.3 (Pin_3); no longer J4.4 (Pin_4), J5.4 (Pin_4), J6.4 (Pin_4), J7.4 (Pin_4)
- net f: now also J4.2 (Pin_2), J5.2 (Pin_2), J6.2 (Pin_2), J7.2 (Pin_2); no longer J4.3 (Pin_3), J5.3 (Pin_3), J6.3 (Pin_3), J7.3 (Pin_3)
- net g: now also J4.1 (Pin_1), J5.1 (Pin_1), J6.1 (Pin_1), J7.1 (Pin_1); no longer J4.2 (Pin_2), J5.2 (Pin_2), J6.2 (Pin_2), J7.2 (Pin_2)
- net g1: now also U1.13 (PB1); no longer U1.10 (PD6)
- net g2: now also U1.12 (PB0); no longer U1.11 (PD7)
- net g3: now also U1.11 (PD7); no longer U1.12 (PB0)
- net g4: now also U1.10 (PD6); no longer U1.13 (PB1)
- net miso: now also J1.2 (Pin_2)
- net mosi: now also J1.3 (Pin_3)
- net reset: now also J1.5 (Pin_5), SW1.1
- net sck: now also J1.4 (Pin_4)
- net at U3.1 (I1): now also U1.32 (PD2); no longer U1.23 (PC0)
- net at U3.10 (O7): now also R2.2; no longer R8.2
- net at U3.11 (O6): now also R3.2; no longer R7.2
- net at U3.12 (O5): now also R4.2; no longer R6.2
- net at U3.14 (O3): now also R6.2; no longer R4.2
- net at U3.15 (O2): now also R7.2; no longer R3.2
- net at U3.16 (O1): now also R8.2; no longer R2.2
- net at U3.2 (I2): now also U1.28 (PC5); no longer U1.24 (PC1)
- net at U3.3 (I3): now also U1.27 (PC4); no longer U1.25 (PC2)
- net at U3.5 (I5): now also U1.25 (PC2); no longer U1.27 (PC4)
- net at U3.6 (I6): now also U1.24 (PC1); no longer U1.28 (PC5)
- net at U3.7 (I7): now also U1.23 (PC0); no longer U1.32 (PD2)
Other:
- moved on the sheet: J4, J5, J6, J7, U3
